Commit message: base_footprintを付記

File: urdf/ std_rover.urdf (robot description, URDF)
Before this commit: robot two_wheeled_robot, 6 links, 5 joints
Links:
- added link base_footprint, mass 0.001
Joints:
- added joint base_footprint_joint: type fixed, parent base_footprint, child base_link, origin xyz=0 0 0 rpy=0 0 0
