Commit message: revise urdf

File: ros2_raspi_rover_description/src/description/ros2_raspi_rover_description.urdf (robot description, URDF)
Before this commit: robot two_wheeled_robot, 7 links, 6 joints
Links:
- link base_link: geometry collision box size=0.11 0.08 0.1; visual box size=0.11 0.08 0.1

Commit message: ロボットが水平じゃなかったので修正

File: ros2_raspi_rover_description/src/description/ros2_raspi_rover_description.urdf (robot description, URDF)
Before this commit: robot two_wheeled_robot, 7 links, 6 joints
Links:
- link caster_cylinder: geometry collision cylinder length=0.02 radius=0.01; visual cylinder length=0.02 radius=0.01
Joints:
- joint caster_joint: origin xyz=0 0 -0.0125 rpy=0 0 0 -> xyz=0 0 -0.01 rpy=0 0 0
- joint cylinder_joint: origin xyz=0.0375 0 -0.05125 rpy=0 0 0 -> xyz=0.0375 0 -0.06 rpy=0 0 0

File: ros2_raspi_rover_description/src/description/ros2_raspi_rover_description.urdf.xacro (robot description, xacro)
@@ -11,5 +11,5 @@
   <xacro:property name="wheel_mass" value="0.1"/>
   <xacro:property name="wheel_inertia" value="0.0001 0.0 0.0 0.0001 0.0 0.0001"/>
-  <xacro:property name="caster_cylinder_size" value="0.01 0.025"/>
+  <xacro:property name="caster_cylinder_size" value="0.01 0.02"/>
   <xacro:property name="caster_cylinder_mass" value="0.05"/>
   <xacro:property name="caster_cylinder_inertia" value="0.001 0.0001 0.0 0.0 0.0 0.0"/>
@@ -158,5 +158,5 @@
     <parent link="base_link"/>
     <child link="caster_cylinder"/>
-    <origin xyz="0.0375 0 -0.05125" rpy="0 0 0"/>
+    <origin xyz="0.0375 0 -0.06" rpy="0 0 0"/>
     <axis xyz="0 1 0"/>
   </joint>
@@ -164,21 +164,25 @@
     <parent link="caster_cylinder"/>
     <child link="caster"/>
-    <origin xyz="0 0 -0.0125" rpy="0 0 0"/>
+    <origin xyz="0 0 -0.01" rpy="0 0 0"/>
+    <limit lower="-3.14159" upper="3.14159" effort="0.0" velocity="0.0"/>
   </joint>
   <!-- Gazebo plugin for differential drive -->
   <gazebo>
-    <plugin name="differential_drive_controller" filename="libgazebo_ros_diff_drive.so">
-      <legacyMode>false</legacyMode>
-      <alwaysOn>true</alwaysOn>
-      <updateRate>100</updateRate>
-      <leftJoint>left_wheel_joint</leftJoint>
-      <rightJoint>right_wheel_joint</rightJoint>
-      <wheelSeparation>0.0875</wheelSeparation>
-      <wheelDiameter>0.06</wheelDiameter>
+    <plugin name="diff_drive" filename="libgazebo_ros_diff_drive.so">
+      <legacy_mode>false</legacy_mode>
+      <always_on>true</always_on>
+      <left_joint>left_wheel_joint</left_joint>
+      <right_joint>right_wheel_joint</right_joint>
+      <wheel_separation>0.0875</wheel_separation>
+      <wheel_diameter>0.06</wheel_diameter>
       <torque>0.5</torque>
-      <commandTopic>cmd_vel</commandTopic>
-      <odometryTopic>odom</odometryTopic>
-      <odometryFrame>odom</odometryFrame>
-      <robotBaseFrame>base_footprint</robotBaseFrame>
+      <!-- output -->
+      <publish_odom>true</publish_odom>
+      <publish_odom_tf>false</publish_odom_tf>
+      <publish_wheel_tf>false</publish_wheel_tf>
+      <command_topic>cmd_vel</command_topic>
+      <odometry_topic>odom</odometry_topic>
+      <odometry_frame>odom</odometry_frame>
+      <robot_base_frame>base_footprint</robot_base_frame>
     </plugin>
   </gazebo>
@@ -209,5 +213,5 @@
         </noise>
       </ray>
-      <plugin name="gazebo_ros_head" filename="libgazebo_ros_laser.so">
+      <plugin name="gazebo_ros_head" filename="libgazebo_ros_ray_sensor.so">
         <topicName>/scan</topicName>
         <frameName>lidar</frameName>

Commit message: nav2でcostmap作成可能にした

File: ros2_raspi_rover_description/src/description/ros2_raspi_rover_description.urdf (robot description, URDF)
Before this commit: robot two_wheeled_robot, 7 links, 6 joints
Links:
- removed link caster
- removed link caster_cylinder
- removed link left_wheel
- removed link lidar
- removed link right_wheel
- added link front_caster; collision sphere radius=${(wheel_radius+wheel_zoff-(base_height/2))}; visual sphere radius=${(wheel_radius+wheel_zoff-(base_height/2))}
- added link lidar_link, mass 0.1; collision cylinder length=0.02 radius=0.02; visual cylinder length=0.02 radius=0.02
- link base_footprint: mass 0.001 -> None
- link base_link: mass 1 -> None; geometry collision box size=${base_length} ${base_width} ${base_height}; visual box size=${base_length} ${base_width} ${base_height}
Joints:
- removed joint base_footprint_joint
- removed joint cylinder_joint
- removed joint left_wheel_joint
- removed joint right_wheel_joint
- added joint base_joint: type fixed, parent base_link, child base_footprint, origin xyz=0.0 0.0 ${-(wheel_radius+wheel_zoff)} rpy=0 0 0
- joint caster_joint: axis 0 1 0 -> (none); child caster -> front_caster; limit lower=-3.14159 upper=3.14159 effort=0.0 velocity=0.0 -> (none); origin xyz=0 0 -0.01 rpy=0 0 0 -> xyz=${caster_cylinder_xoff} 0.0 ${-(base_height/2)} rpy=0 0 0; parent caster_cylinder -> base_link; type revolute -> fixed
- joint lidar_joint: child lidar -> lidar_link; origin xyz=0 0 0.0625 rpy=0 0 0 -> xyz=0 0 0.062 rpy=0 0 0
